File: Schematic/Main Schematic/SENSOR.kicad_sch (KiCad schematic)
At the start: 11 parts, among them IC1 LM75AD,118

Commit message: Update
Connections:
- net +3V3 renamed 3.3V
Other:
- note added: "Analogue Sensor"
- note added: "Digital Sensor"
Changed lines of the file:
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@@
     (title "Sensors")
     (company "UCT")
-    (comment 4 "Author: Zwivhuya Ndou")
+    (comment 2 "Sensing Module")
+    (comment 3 "Author: Zwivhuya Ndou")
+    (comment 4 "Team 26")
   )
   (junction (at 164.1856 111.379) (diameter 0) (color 0 0 0 0)
@@
   (junction (at 110.6932 125.4506) (diameter 0) (color 0 0 0 0)
   )
-  (junction (at 113.1824 100.0506) (diameter 0) (color 0 0 0 0)
-  )
   (junction (at 113.2332 105.7656) (diameter 0) (color 0 0 0 0)
   )
@@
   (junction (at 180.4416 111.379) (diameter 0) (color 0 0 0 0)
   )
+  (junction (at 113.2332 100.0506) (diameter 0) (color 0 0 0 0)
+  )
   (junction (at 65.6082 125.4506) (diameter 0) (color 0 0 0 0)
   )
@@
     (stroke (width 0) (type default))
   )
-  (wire (pts (xy 110.6932 100.0506) (xy 113.1824 100.0506))
-    (stroke (width 0) (type default))
-  )
   (wire (pts (xy 85.2932 127.9906) (xy 85.2932 132.4356))
     (stroke (width 0) (type default))
@@
     (stroke (width 0) (type default))
   )
+  (wire (pts (xy 113.2332 98.7044) (xy 113.2332 100.0506))
+    (stroke (width 0) (type default))
+  )
+  (wire (pts (xy 70.0532 105.7656) (xy 78.9432 105.7656))
+    (stroke (width 0) (type default))
+  )
+  (polyline (pts (xy 155.956 143.2306) (xy 214.884 143.0782))
+    (stroke (width 0) (type default))
+  )
+  (polyline (pts (xy 156.0068 84.6582) (xy 156.1592 143.5862))
+    (stroke (width 0) (type default))
+  )
+  (wire (pts (xy 110.6932 125.4506) (xy 110.6932 127.9906))
+    (stroke (width 0) (type default))
+  )
+  (wire (pts (xy 70.0532 122.9106) (xy 70.0532 113.3856))
+    (stroke (width 0) (type default))
+  )
+  (polyline (pts (xy 121.4628 83.185) (xy 57.2516 83.5914))
+    (stroke (width 0) (type default))
+  )
   (wire (pts (xy 113.2332 100.0506) (xy 113.2332 105.7656))
     (stroke (width 0) (type default))
   )
-  (wire (pts (xy 70.0532 105.7656) (xy 78.9432 105.7656))
-    (stroke (width 0) (type default))
-  )
-  (polyline (pts (xy 155.956 143.2306) (xy 214.884 143.0782))
-    (stroke (width 0) (type default))
-  )
-  (polyline (pts (xy 156.0068 84.6582) (xy 156.1592 143.5862))
-    (stroke (width 0) (type default))
-  )
-  (wire (pts (xy 110.6932 125.4506) (xy 110.6932 127.9906))
-    (stroke (width 0) (type default))
-  )
-  (wire (pts (xy 70.0532 122.9106) (xy 70.0532 113.3856))
-    (stroke (width 0) (type default))
-  )
-  (polyline (pts (xy 121.4628 83.185) (xy 57.2516 83.5914))
-    (stroke (width 0) (type default))
-  )
-  (wire (pts (xy 113.1824 92.4306) (xy 113.1824 100.0506))
-    (stroke (width 0) (type default))
-  )
   (wire (pts (xy 85.2932 120.3706) (xy 82.1182 120.3706))
     (stroke (width 0) (type default))
@@
     (stroke (width 0) (type default))
   )
-  (wire (pts (xy 113.1824 100.0506) (xy 113.2332 100.0506))
+  (wire (pts (xy 110.6932 100.0506) (xy 113.2332 100.0506))
     (stroke (width 0) (type default))
   )
@@
     (effects (font (size 1.27 1.27)) (justify left bottom))
   )
+  (text "Analogue Sensor\n" (at 169.926 147.4216 0)
+    (effects (font (size 3 3) (thickness 0.6) bold) (justify left bottom))
+  )
   (text "Set internal ADC to connect PB0\n\n" (at 173.0756 110.2614 0)
     (effects (font (size 1.27 1.27)) (justify left bottom))
+  )
+  (text "Digital Sensor\n" (at 73.914 147.1676 0)
+    (effects (font (size 3 3) bold) (justify left bottom))
   )
   (text "TEMPERATURE SENSOR" (at 87.8332 110.2106 0)
@@
     (effects (font (size 1.27 1.27)) (justify left bottom))
   )
+  (hierarchical_label "3.3V" (shape input) (at 113.2332 98.7044 0) (fields_autoplaced)
+    (effects (font (size 1.27 1.27)) (justify left))
+  )
   (hierarchical_label "LDR" (shape input) (at 202.2856 111.379 0) (fields_autoplaced)
+    (effects (font (size 1.27 1.27)) (justify left))
+  )
+  (hierarchical_label "3.3V" (shape input) (at 164.1856 97.1804 0) (fields_autoplaced)
     (effects (font (size 1.27 1.27)) (justify left))
   )
@@
     )
   )
-  (symbol (lib_id "power:+3V3") (at 113.1824 92.4306 0) (unit 1)
-    (in_bom yes) (on_board yes) (dnp no) (fields_autoplaced)
-    (property "Reference" "#PWR012" (at 113.1824 96.2406 0)
-      (effects (font (size 1.27 1.27)) hide)
-    )
-    (property "Value" "+3V3" (at 113.1824 89.1794 0)
-      (effects (font (size 1.27 1.27)))
-    )
-    (property "Footprint" "" (at 113.1824 92.4306 0)
-      (effects (font (size 1.27 1.27)) hide)
-    )
-    (property "Datasheet" "" (at 113.1824 92.4306 0)
-      (effects (font (size 1.27 1.27)) hide)
-    )
-    (pin "1")
-    (instances
-      (project "Main Schematic"
-        (path "/81c41bad-bb43-41af-b405-18d135a809b1/820a1ce6-42c1-4792-8ad0-5e2a5c074ed4"
-          (reference "#PWR012") (unit 1)
-        )
-      )
-    )
-  )
   (symbol (lib_id "Device:R") (at 70.0532 109.5756 0) (unit 1)
     (in_bom yes) (on_board yes) (dnp no) (fields_autoplaced)
@@
         )
       )
-    )
-  )
-  (symbol (lib_id "power:+3V3") (at 164.1856 97.1804 0) (unit 1)
-    (in_bom yes) (on_board yes) (dnp no) (fields_autoplaced)
-    (property "Reference" "#PWR014" (at 164.1856 100.9904 0)
-      (effects (font (size 1.27 1.27)) hide)
-    )
-    (property "Value" "+3V3" (at 164.1856 93.9292 0)
-      (effects (font (size 1.27 1.27)))
-    )
-    (property "Footprint" "" (at 164.1856 97.1804 0)
-      (effects (font (size 1.27 1.27)) hide)
-    )
-    (property "Datasheet" "" (at 164.1856 97.1804 0)
-      (effects (font (size 1.27 1.27)) hide)
-    )
-    (pin "1")
-    (instances
-      (project "Main Schematic"
-        (path "/81c41bad-bb43-41af-b405-18d135a809b1/820a1ce6-42c1-4792-8ad0-5e2a5c074ed4"
-          (reference "#PWR014") (unit 1)
-        )
-      )
