File: Schematic/Main Schematic/MCU.kicad_sch (KiCad schematic)
At the start: 10 parts, among them J1 Conn_ARM_JTAG_SWD_10, J11 Conn_01x02_Male, SW1 SW_Push, U1 STM32F051C6Tx, U3 CH340C

Commit message: Updated main schematic but not entirely
Parts:
- removed J1: Conn_ARM_JTAG_SWD_10, symbol Connector:Conn_ARM_JTAG_SWD_10
- renumbered R3 to R12, R2 to R13, U1 to U4
Other:
- moved on the sheet: J11
Changed lines of the file:
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@@
     (stroke (width 0) (type default))
   )
-  (wire (pts (xy 205.74 87.63) (xy 205.74 88.9))
+  (wire (pts (xy 232.41 93.98) (xy 232.41 95.25))
     (stroke (width 0) (type default))
   )
@@
     (stroke (width 0) (type default))
   )
-  (wire (pts (xy 195.58 120.65) (xy 204.47 120.65))
-    (stroke (width 0) (type default))
-  )
   (wire (pts (xy 219.71 62.23) (xy 213.36 62.23))
     (stroke (width 0) (type default))
@@
     (stroke (width 0) (type default))
   )
-  (wire (pts (xy 182.88 92.71) (xy 182.88 105.41))
-    (stroke (width 0) (type default))
-  )
-  (wire (pts (xy 195.58 118.11) (xy 204.47 118.11))
-    (stroke (width 0) (type default))
-  )
-  (wire (pts (xy 182.88 135.89) (xy 182.88 140.97))
-    (stroke (width 0) (type default))
-  )
   (wire (pts (xy 140.97 72.39) (xy 152.4 72.39))
     (stroke (width 0) (type default))
@@
     (stroke (width 0) (type default))
   )
-  (wire (pts (xy 207.01 91.44) (xy 203.2 91.44))
+  (wire (pts (xy 233.68 97.79) (xy 229.87 97.79))
     (stroke (width 0) (type default))
   )
@@
     (stroke (width 0) (type default))
   )
-  (wire (pts (xy 205.74 88.9) (xy 203.2 88.9))
+  (wire (pts (xy 232.41 95.25) (xy 229.87 95.25))
     (stroke (width 0) (type default))
   )
@@
     (stroke (width 0) (type default))
   )
-  (wire (pts (xy 207.01 87.63) (xy 205.74 87.63))
+  (wire (pts (xy 233.68 93.98) (xy 232.41 93.98))
     (stroke (width 0) (type default))
   )
@@
   )
   (wire (pts (xy 123.19 50.8) (xy 123.19 57.15))
-    (stroke (width 0) (type default))
-  )
-  (wire (pts (xy 195.58 113.03) (xy 204.47 113.03))
     (stroke (width 0) (type default))
   )
@@
     (effects (font (size 1.27 1.27)) (justify left bottom))
   )
-  (label "debugger" (at 186.69 135.89 0) (fields_autoplaced)
-    (effects (font (size 1.27 1.27)) (justify left bottom))
-  )
   (label "3V3" (at 123.19 50.8 270) (fields_autoplaced)
     (effects (font (size 1.27 1.27)) (justify right bottom))
@@
     (effects (font (size 1.27 1.27)) (justify right bottom))
   )
-  (label "T_SWDIO" (at 204.47 120.65 0) (fields_autoplaced)
-    (effects (font (size 1.27 1.27)) (justify left bottom))
-  )
-  (label "T_SWCLK" (at 204.47 118.11 0) (fields_autoplaced)
-    (effects (font (size 1.27 1.27)) (justify left bottom))
-  )
   (label "3V3" (at 128.27 50.8 270) (fields_autoplaced)
     (effects (font (size 1.27 1.27)) (justify right bottom))
-  )
-  (label "NRST" (at 204.47 113.03 0) (fields_autoplaced)
-    (effects (font (size 1.27 1.27)) (justify left bottom))
   )
   (label "GND" (at 125.73 146.05 90) (fields_autoplaced)
@@
     )
   )
-  (global_label "USB-" (shape input) (at 207.01 91.44 0) (fields_autoplaced)
+  (global_label "USB-" (shape input) (at 233.68 97.79 0) (fields_autoplaced)
     (effects (font (size 1.27 1.27)) (justify left))
-    (property "Intersheetrefs" "${INTERSHEET_REFS}" (at 214.8055 91.3606 0)
+    (property "Intersheetrefs" "${INTERSHEET_REFS}" (at 241.4755 97.7106 0)
       (effects (font (size 1.27 1.27)) (justify left) hide)
     )
@@
     )
   )
-  (global_label "USB+" (shape input) (at 207.01 87.63 0) (fields_autoplaced)
+  (global_label "USB+" (shape input) (at 233.68 93.98 0) (fields_autoplaced)
     (effects (font (size 1.27 1.27)) (justify left))
-    (property "Intersheetrefs" "${INTERSHEET_REFS}" (at 214.8055 87.5506 0)
+    (property "Intersheetrefs" "${INTERSHEET_REFS}" (at 241.4755 93.9006 0)
       (effects (font (size 1.27 1.27)) (justify left) hide)
     )
@@
   (symbol (lib_id "Device:R_US") (at 165.1 46.99 0) (unit 1)
     (in_bom yes) (on_board yes) (dnp no) (fields_autoplaced)
-    (property "Reference" "R2" (at 167.64 46.355 0)
+    (property "Reference" "R13" (at 167.64 46.355 0)
       (effects (font (size 1.27 1.27)) (justify left))
     )
@@
   (symbol (lib_id "power:GND") (at 63.5 39.37 0) (unit 1)
     (in_bom yes) (on_board yes) (dnp no) (fields_autoplaced)
-    (property "Reference" "#PWR03" (at 63.5 45.72 0)
+    (property "Reference" "#PWR014" (at 63.5 45.72 0)
       (effects (font (size 1.27 1.27)) hide)
     )
@@
   (symbol (lib_id "Device:R_US") (at 81.28 55.88 180) (unit 1)
     (in_bom yes) (on_board yes) (dnp no) (fields_autoplaced)
-    (property "Reference" "R3" (at 83.82 55.245 0)
+    (property "Reference" "R12" (at 83.82 55.245 0)
       (effects (font (size 1.27 1.27)) (justify right))
     )
@@
   (symbol (lib_id "power:+3V3") (at 165.1 36.83 0) (unit 1)
     (in_bom yes) (on_board yes) (dnp no) (fields_autoplaced)
-    (property "Reference" "#PWR02" (at 165.1 40.64 0)
+    (property "Reference" "#PWR016" (at 165.1 40.64 0)
       (effects (font (size 1.27 1.27)) hide)
     )
@@
     )
   )
-  (symbol (lib_id "power:+3V3") (at 182.88 92.71 0) (unit 1)
-    (in_bom yes) (on_board yes) (dnp no) (fields_autoplaced)
-    (property "Reference" "#PWR06" (at 182.88 96.52 0)
-      (effects (font (size 1.27 1.27)) hide)
-    )
-    (property "Value" "+3V3" (at 182.88 88.9 0)
-      (effects (font (size 1.27 1.27)))
-    )
-    (property "Footprint" "" (at 182.88 92.71 0)
-      (effects (font (size 1.27 1.27)) hide)
-    )
-    (property "Datasheet" "" (at 182.88 92.71 0)
-      (effects (font (size 1.27 1.27)) hide)
-    )
-    (pin "1")
-    (instances
-      (project "Main Schematic"
-        (path "/81c41bad-bb43-41af-b405-18d135a809b1/ae15d31d-f7b4-4051-b9d0-3a01939afe0e"
-          (reference "#PWR017") (unit 1)
-        )
-      )
-      (project "Microcontroller Design"
-        (path "/b8d97438-63f4-433e-afdc-8e43ab7e4842"
-          (reference "#PWR06") (unit 1)
-        )
-      )
-      (project "MCU"
-        (path "/e0666d22-e687-4adb-b95b-6588526d91f1"
-          (reference "#PWR07") (unit 1)
-        )
-      )
-    )
-  )
-  (symbol (lib_id "Connector:Conn_01x02_Male") (at 198.12 88.9 0) (unit 1)
-    (in_bom yes) (on_board yes) (dnp no) (fields_autoplaced)
-    (property "Reference" "J11" (at 198.755 83.185 0)
-      (effects (font (size 1.27 1.27)))
-    )
-    (property "Value" "Conn_01x02_Male" (at 198.755 85.725 0)
-      (effects (font (size 1.27 1.27)))
-    )
-    (property "Footprint" "Connector_PinHeader_2.54mm:PinHeader_1x02_P2.54mm_Vertical" (at 198.12 88.9 0)
-      (effects (font (size 1.27 1.27)) hide)
-    )
-    (property "Datasheet" "~" (at 198.12 88.9 0)
+  (symbol (lib_id "Connector:Conn_01x02_Male") (at 224.79 95.25 0) (unit 1)
+    (in_bom yes) (on_board yes) (dnp no) (fields_autoplaced)
+    (property "Reference" "J11" (at 225.425 89.535 0)
+      (effects (font (size 1.27 1.27)))
+    )
+    (property "Value" "Conn_01x02_Male" (at 225.425 92.075 0)
+      (effects (font (size 1.27 1.27)))
+    )
+    (property "Footprint" "Connector_PinHeader_2.54mm:PinHeader_1x02_P2.54mm_Vertical" (at 224.79 95.25 0)
+      (effects (font (size 1.27 1.27)) hide)
+    )
+    (property "Datasheet" "~" (at 224.79 95.25 0)
       (effects (font (size 1.27 1.27)) hide)
     )
@@
     )
   )
-  (symbol (lib_id "power:GND") (at 182.88 140.97 0) (unit 1)
-    (in_bom yes) (on_board yes) (dnp no) (fields_autoplaced)
-    (property "Reference" "#PWR07" (at 182.88 147.32 0)
-      (effects (font (size 1.27 1.27)) hide)
-    )
-    (property "Value" "GND" (at 182.88 146.05 0)
-      (effects (font (size 1.27 1.27)))
-    )
-    (property "Footprint" "" (at 182.88 140.97 0)
-      (effects (font (size 1.27 1.27)) hide)
-    )
-    (property "Datasheet" "" (at 182.88 140.97 0)
-      (effects (font (size 1.27 1.27)) hide)
-    )
-    (pin "1")
-    (instances
-      (project "Main Schematic"
-        (path "/81c41bad-bb43-41af-b405-18d135a809b1/ae15d31d-f7b4-4051-b9d0-3a01939afe0e"
-          (reference "#PWR018") (unit 1)
-        )
-      )
-      (project "Microcontroller Design"
-        (path "/b8d97438-63f4-433e-afdc-8e43ab7e4842"
-          (reference "#PWR07") (unit 1)
-        )
-      )
-      (project "MCU"
-        (path "/e0666d22-e687-4adb-b95b-6588526d91f1"
-          (reference "#PWR08") (unit 1)
-        )
-      )
-    )
-  )
   (symbol (lib_id "power:GND") (at 81.28 59.69 0) (unit 1)
     (in_bom yes) (on_board yes) (dnp no) (fields_autoplaced)
-    (property "Reference" "#PWR04" (at 81.28 66.04 0)
+    (property "Reference" "#PWR015" (at 81.28 66.04 0)
       (effects (font (size 1.27 1.27)) hide)
     )
@@
   (symbol (lib_id "MCU_ST_STM32F0:STM32F051C6Tx") (at 125.73 100.33 0) (unit 1)
     (in_bom yes) (on_board yes) (dnp no) (fields_autoplaced)
-    (property "Reference" "U1" (at 130.2259 140.97 0)
+    (property "Reference" "U4" (at 130.2259 140.97 0)
       (effects (font (size 1.27 1.27)) (justify left))
     )
@@
         )
       )
-    )
-  )
-  (symbol (lib_id "Connector:Conn_ARM_JTAG_SWD_10") (at 182.88 120.65 0) (unit 1)
-    (in_bom yes) (on_board yes) (dnp no) (fields_autoplaced)
-    (property "Reference" "J1" (at 171.45 120.015 0)
-      (effects (font (size 1.27 1.27)) (justify right))
-    )
-    (property "Value" "Conn_ARM_JTAG_SWD_10" (at 171.45 122.555 0)
-      (effects (font (size 1.27 1.27)) (justify right))
-    )
-    (property "Footprint" "" (at 182.88 120.65 0)
-      (effects (font (size 1.27 1.27)) hide)
-    )
-    (property "Datasheet" "http://infocenter.arm.com/help/topic/com.arm.doc.ddi0314h/DDI0314H_coresight_components_trm.pdf" (at 173.99 152.4 90)
-      (effects (font (size 1.27 1.27)) hide)
-    )
-    (pin "1")
-    (pin "10")
-    (pin "2")
-    (pin "3")
-    (pin "4")
-    (pin "5")
-    (pin "6")
-    (pin "7")
-    (pin "8")
-    (pin "9")
-    (instances
-      (project "Main Schematic"
-        (path "/81c41bad-bb43-41af-b405-18d135a809b1/ae15d31d-f7b4-4051-b9d0-3a01939afe0e"
-          (reference "J2") (unit 1)
-        )
-      )
-      (project "Microcontroller Design"
-        (path "/b8d97438-63f4-433e-afdc-8e43ab7e4842"
-          (reference "J1") (unit 1)
-        )
-      )
-      (project "MCU"
-        (path "/e0666d22-e687-4adb-b95b-6588526d91f1"
-          (reference "J3") (unit 1)
-        )
-      )

Commit message: 'MCU.kicad_sch'
Parts:
- removed J11: Conn_01x02_Male, Connector_PinHeader_2.54mm:PinHeader_1x02_P2.54mm_Vertical, symbol Connector:Conn_01x02_Male
- removed TP8: TXD, TestPoint:TestPoint_Pad_1.0x1.0mm, symbol Connector:TestPoint
- removed TP9: RXD, TestPoint:TestPoint_Pad_1.0x1.0mm, symbol Connector:TestPoint
- added C11: 10nF, CAP_10NF:CAPC1005X55N, symbol Device:C
- added TP5: SDA2, TestPoint:TestPoint_Pad_1.0x1.0mm, symbol Connector:TestPoint
- added U6: M24C16-RMN6TP, M24:SOIC127P600X175-8N, symbol M24C16-RMN6TP:M24C16-RMN6TP
Connections:
- net GND: now also C11.2, U6.1 (E0), U6.2 (E1), U6.3 (E2), U6.4 (VSS)
- net at C7.1, U3.16 (VCC): no longer U3.4 (V3)
- new net SCL2: U6.6 (SCL)
- new net SDA2: TP5.1, U6.5 (SDA)
- new net V_out: C11.1, U3.4 (V3), U6.8 (VCC)
- new net Write1: U6.7 (~{WC})
Other:
- note added: "EEPROM"
- title: (none) -> Microcontroller Interface
- moved on the sheet: C7, R12, R13, SW1, U3, U4

Commit message: 'Updated'
Parts:
- removed R12: 10k, symbol Device:R_US
- removed R13: 4k7, symbol Device:R_US
- removed SW1: SW_Push, symbol Switch:SW_Push
- removed U4: STM32F051C6Tx, Package_QFP:LQFP-48_7x7mm_P0.5mm, symbol MCU_ST_STM32F0:STM32F051C6Tx
- added J5: Conn_01x02_Pin, symbol Connector:Conn_01x02_Pin
- added TP1: Vout, TestPoint:TestPoint_Pad_1.0x1.0mm, symbol Connector:TestPoint
- added TP2: SCL2, TestPoint:TestPoint_Pad_1.0x1.0mm, symbol Connector:TestPoint
- added TP3, TP5, TP6, TP7: ~, TestPoint:TestPoint_Pad_1.0x1.0mm, symbol Connector:TestPoint
- renumbered TP5 to TP
Connections:
- net USB- is gone; now on net USB D+: U3.6 (UD-)
- net RXD: now also TP3.1
- net SCL2: now also TP2.1
- net TXD: now also TP5.1
- net V_out: now also TP1.1
- net USB+ renamed USB D+
- net USB D+: now also TP6.1, TP7.1
- new net USB +: J5.1 (Pin_1)
- new net USB D-: J5.2 (Pin_2)
Other:
- note added: "- Used to stored data collected from the sensing module - Pin 5(SCL2) and pin 6(SDA2) will connect to STM32F051C6"
- note added: "Sub-circuit is used to convert USB to UART via the TXD and RXD pins of the CH340C C10 actS as decoupling capacitors to filter out noise on the lines. All unused pins are not connected. Test points to be added for debugging purposes"
- note removed: "MICROCONTROLLER"
- moved on the sheet: C11, C7, U3, U6

Commit message: 'Updated'
Parts:
- TP1: value Vout -> Testing Point
- TP3, TP5, TP6: value ~ -> ~TP
Other:
- note added: "- Used to stored data collected from the sensing module - Pin 5(SCL2) and pin 6(SDA2) will connect to STM32F051C6 - Pin 7(WC), will connect to MCU for prevention of write operations"
- note added: "circuit is used to convert USB to UART via the TXD and RXD pins of the CH340C C10 actS as decoupling capacitors to filter out noise on the lines. All unused pins are not connected. Test points to be added for debugging purposes"
- note removed: "- Used to stored data collected from the sensing module - Pin 5(SCL2) and pin 6(SDA2) will connect to STM32F051C6"
- note removed: "Sub-circuit is used to convert USB to UART via the TXD and RXD pins of the CH340C C10 actS as decoupling capacitors to filter out noise on the lines. All unused pins are not connected. Test points to be added for debugging purposes"
Changed lines of the file:
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@@
     (effects (font (size 1.27 1.27) (color 140 0 0 1)) (justify left bottom))
   )
-  (text "Sub-circuit is used to convert USB to UART via the TXD and RXD pins of the CH340C\nC10 actS as decoupling capacitors to filter out noise on the lines.\nAll unused pins are not connected. Test points to be added for debugging purposes"
+  (text "circuit is used to convert USB to UART via the TXD and RXD pins of the CH340C\nC10 actS as decoupling capacitors to filter out noise on the lines.\nAll unused pins are not connected. Test points to be added for debugging purposes\n"
     (at 52.07 30.48 0)
     (effects (font (face "KiCad Font") (size 1.5 1.5)) (justify left bottom))
@@
     (effects (font (size 2 2) (thickness 0.4) bold) (justify left bottom))
   )
-  (text "- Used to stored data collected from the sensing module\n- Pin 5(SCL2) and pin 6(SDA2) will connect to STM32F051C6\n"
-    (at 149.86 34.29 0)
+  (text "- Used to stored data collected from the sensing module\n- Pin 5(SCL2) and pin 6(SDA2) will connect to STM32F051C6\n- Pin 7(WC), will connect to MCU for prevention of write operations\n\n"
+    (at 149.86 36.83 0)
     (effects (font (size 1.27 1.27)) (justify left bottom))
   )
@@
       (effects (font (size 1.27 1.27)) (justify left) hide)
     )
-    (property "Value" "~" (at 49.53 57.277 0)
+    (property "Value" "~TP" (at 49.53 57.277 0)
       (effects (font (size 1.27 1.27)) (justify left))
     )
@@
       (effects (font (size 1.27 1.27)) (justify left) hide)
     )
-    (property "Value" "~" (at 54.61 49.403 0)
+    (property "Value" "~TP" (at 54.61 49.403 0)
       (effects (font (size 1.27 1.27)) (justify left))
     )
@@
       (effects (font (size 1.27 1.27)) hide)
     )
+    (property "Field4" "" (at 52.07 52.07 90)
+      (effects (font (size 1.27 1.27)) hide)
+    )
     (pin "1")
     (instances
@@
       (effects (font (size 1.27 1.27)) (justify left) hide)
     )
-    (property "Value" "~" (at 96.52 57.277 0)
+    (property "Value" "~TP" (at 96.52 57.277 0)
       (effects (font (size 1.27 1.27)) (justify left))
     )
@@
       (effects (font (size 1.27 1.27)) (justify left) hide)
     )
-    (property "Value" "Vout" (at 243.84 57.023 0)
-      (effects (font (size 1.27 1.27)) (justify left))
-    )
+    (property "Value" "Testing Point" (at 243.84 57.023 0)
+      (effects (font (size 1.27 1.27)) (justify left))
+    )
