File: Schematic/Main Schematic/MCU.kicad_sch (KiCad schematic)
At the start: 10 parts, among them J7 Conn_01x02_Pin, U4 M24C16-RMN6TP

Commit message: Edit
Connections:
- net RXD: now also TP7.1; no longer TP6.1
- net TXD: now also TP6.1; no longer TP7.1
Changed lines of the file:
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@@
   (junction (at 94.5388 44.45) (diameter 0) (color 0 0 0 0)
   )
+  (junction (at 241.3 59.69) (diameter 0) (color 0 0 0 0)
+  )
+  (junction (at 50.8 54.61) (diameter 0) (color 0 0 0 0)
+  )
   (junction (at 52.07 52.07) (diameter 0) (color 0 0 0 0)
-  )
-  (junction (at 241.3 59.69) (diameter 0) (color 0 0 0 0)
-  )
-  (junction (at 52.07 54.61) (diameter 0) (color 0 0 0 0)
   )
   (no_connect (at 63.5 67.31))
@@
     (stroke (width 0) (type default))
   )
-  (wire (pts (xy 45.72 54.61) (xy 52.07 54.61))
-    (stroke (width 0) (type default))
-  )
   (polyline (pts (xy 148.59 96.52) (xy 148.59 21.59))
     (stroke (width 0) (type default))
   )
+  (wire (pts (xy 52.07 52.07) (xy 63.5 52.07))
+    (stroke (width 0) (type default))
+  )
   (wire (pts (xy 200.66 57.15) (xy 200.66 59.69))
     (stroke (width 0) (type default))
@@
     (stroke (width 0) (type default))
   )
+  (wire (pts (xy 50.8 54.61) (xy 63.5 54.61))
+    (stroke (width 0) (type default))
+  )
   (wire (pts (xy 191.77 57.15) (xy 200.66 57.15))
     (stroke (width 0) (type default))
@@
     (stroke (width 0) (type default))
   )
-  (wire (pts (xy 52.07 54.61) (xy 63.5 54.61))
+  (wire (pts (xy 45.72 54.61) (xy 50.8 54.61))
     (stroke (width 0) (type default))
   )
@@
   )
   (polyline (pts (xy 24.13 96.52) (xy 24.13 21.59))
-    (stroke (width 0) (type default))
-  )
-  (wire (pts (xy 52.07 52.07) (xy 63.5 52.07))
     (stroke (width 0) (type default))
   )
@@
     )
   )
-  (symbol (lib_id "Connector:TestPoint") (at 52.07 54.61 180) (unit 1)
-    (in_bom yes) (on_board yes) (dnp no) (fields_autoplaced)
-    (property "Reference" "TP7" (at 53.3401 59.69 90)
+  (symbol (lib_id "Connector:TestPoint") (at 52.07 52.07 0) (unit 1)
+    (in_bom yes) (on_board yes) (dnp no) (fields_autoplaced)
+    (property "Reference" "TP7" (at 50.7999 46.99 90)
       (effects (font (size 1.27 1.27)) (justify left) hide)
     )
-    (property "Value" "TXD testpoint" (at 54.61 58.547 0)
-      (effects (font (size 1.27 1.27)) (justify right))
-    )
-    (property "Footprint" "TestPoint:TestPoint_Pad_1.0x1.0mm" (at 46.99 54.61 0)
-      (effects (font (size 1.27 1.27)) hide)
-    )
-    (property "Datasheet" "~" (at 46.99 54.61 0)
+    (property "Value" "TXD testpoint" (at 53.4924 49.403 0)
+      (effects (font (size 1.27 1.27)) (justify left))
+    )
+    (property "Footprint" "TestPoint:TestPoint_Pad_1.0x1.0mm" (at 57.15 52.07 0)
+      (effects (font (size 1.27 1.27)) hide)
+    )
+    (property "Datasheet" "~" (at 57.15 52.07 0)
       (effects (font (size 1.27 1.27)) hide)
     )
@@
     )
   )
-  (symbol (lib_id "Connector:TestPoint") (at 52.07 52.07 0) (unit 1)
-    (in_bom yes) (on_board yes) (dnp no) (fields_autoplaced)
-    (property "Reference" "TP6" (at 50.7999 46.99 90)
+  (symbol (lib_id "Connector:TestPoint") (at 50.8 54.61 180) (unit 1)
+    (in_bom yes) (on_board yes) (dnp no) (fields_autoplaced)
+    (property "Reference" "TP6" (at 52.0701 59.69 90)
       (effects (font (size 1.27 1.27)) (justify left) hide)
     )
-    (property "Value" "RXD testpoint" (at 54.61 49.403 0)
-      (effects (font (size 1.27 1.27)) (justify left))
-    )
-    (property "Footprint" "TestPoint:TestPoint_Pad_1.0x1.0mm" (at 57.15 52.07 0)
-      (effects (font (size 1.27 1.27)) hide)
-    )
-    (property "Datasheet" "~" (at 57.15 52.07 0)
-      (effects (font (size 1.27 1.27)) hide)
-    )
-    (property "Field4" "" (at 52.07 52.07 90)
-      (effects (font (size 1.27 1.27)) hide)
-    )
+    (property "Value" "RXD testpoint" (at 53.0352 58.547 0)
+      (effects (font (size 1.27 1.27)) (justify right))
+    )
+    (property "Footprint" "TestPoint:TestPoint_Pad_1.0x1.0mm" (at 45.72 54.61 0)
+      (effects (font (size 1.27 1.27)) hide)
+    )
+    (property "Datasheet" "~" (at 45.72 54.61 0)
+      (effects (font (size 1.27 1.27)) hide)
+    )
+    (property "Field4" "" (at 50.8 54.61 90)
+      (effects (font (size 1.27 1.27)) hide)
+    )
